File: probatio_base.brd (EAGLE design)
At the start: 50 x 50 mm, 13 parts

Commit message: longer smd pads and no drills
Parts:
- moved U$13 2.40 mm to (24.9, 24.2)
- moved U$12 0.63 mm to (48.1, 9.00)
- moved U$5 0.63 mm to (9.00, 48.1)
- moved U$6 0.63 mm to (41.0, 48.1)
- moved U$7 0.63 mm to (48.1, 41.0)
- moved U$10 0.63 mm to (9.00, 1.91)
- moved U$11 0.63 mm to (41.0, 1.91)
- moved U$8 0.63 mm to (1.91, 41.0)
- moved U$9 0.63 mm to (1.91, 9.00)
Routing:
- net VCC: track 198.7 -> 203.7 mm
- net GND: track 169.1 -> 174.1 mm
- net SDA: track 202.4 -> 207.5 mm
- net SCL: track 205.2 -> 209.5 mm
Other:
- board text added: "base-pcb v0_3_2"
- board text removed: "base-pcb v0_3_1"

Commit message: probatio logo
Parts:
- added U$14: (no value), Batebit:PROBATIO
- moved U$13 2.40 mm to (25.0, 26.6)
Other:
- board text removed: "probatio"
Changed lines of the file:
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@@
 <layer number="14" name="Route14" color="1" fill="6" visible="no" active="no"/>
 <layer number="15" name="Route15" color="4" fill="6" visible="no" active="no"/>
-<layer number="16" name="Bottom" color="1" fill="1" visible="yes" active="yes"/>
+<layer number="16" name="Bottom" color="1" fill="1" visible="no" active="yes"/>
 <layer number="17" name="Pads" color="2" fill="1" visible="yes" active="yes"/>
 <layer number="18" name="Vias" color="2" fill="1" visible="yes" active="yes"/>
@@
 <layer number="20" name="Dimension" color="15" fill="1" visible="yes" active="yes"/>
 <layer number="21" name="tPlace" color="7" fill="1" visible="yes" active="yes"/>
-<layer number="22" name="bPlace" color="7" fill="1" visible="yes" active="yes"/>
+<layer number="22" name="bPlace" color="7" fill="1" visible="no" active="yes"/>
 <layer number="23" name="tOrigins" color="15" fill="1" visible="yes" active="yes"/>
-<layer number="24" name="bOrigins" color="15" fill="1" visible="yes" active="yes"/>
+<layer number="24" name="bOrigins" color="15" fill="1" visible="no" active="yes"/>
 <layer number="25" name="tNames" color="7" fill="1" visible="yes" active="yes"/>
-<layer number="26" name="bNames" color="7" fill="1" visible="yes" active="yes"/>
+<layer number="26" name="bNames" color="7" fill="1" visible="no" active="yes"/>
 <layer number="27" name="tValues" color="7" fill="1" visible="no" active="yes"/>
 <layer number="28" name="bValues" color="7" fill="1" visible="no" active="yes"/>
@@
 <layer number="38" name="bTest" color="7" fill="1" visible="no" active="yes"/>
 <layer number="39" name="tKeepout" color="4" fill="11" visible="yes" active="yes"/>
-<layer number="40" name="bKeepout" color="1" fill="11" visible="yes" active="yes"/>
+<layer number="40" name="bKeepout" color="1" fill="11" visible="no" active="yes"/>
 <layer number="41" name="tRestrict" color="4" fill="10" visible="yes" active="yes"/>
-<layer number="42" name="bRestrict" color="1" fill="10" visible="yes" active="yes"/>
+<layer number="42" name="bRestrict" color="1" fill="10" visible="no" active="yes"/>
 <layer number="43" name="vRestrict" color="2" fill="10" visible="no" active="yes"/>
 <layer number="44" name="Drills" color="7" fill="1" visible="no" active="yes"/>
-<layer number="45" name="Holes" color="7" fill="1" visible="yes" active="yes"/>
+<layer number="45" name="Holes" color="7" fill="1" visible="no" active="yes"/>
 <layer number="46" name="Milling" color="3" fill="1" visible="no" active="yes"/>
 <layer number="47" name="Measures" color="7" fill="1" visible="no" active="yes"/>
@@
 <layer number="50" name="dxf" color="7" fill="1" visible="no" active="no"/>
 <layer number="51" name="tDocu" color="7" fill="1" visible="yes" active="yes"/>
-<layer number="52" name="bDocu" color="7" fill="1" visible="yes" active="yes"/>
+<layer number="52" name="bDocu" color="7" fill="1" visible="no" active="yes"/>
 <layer number="53" name="tGND_GNDA" color="7" fill="9" visible="no" active="no"/>
 <layer number="54" name="bGND_GNDA" color="1" fill="9" visible="no" active="no"/>
@@
 <wire x1="49" y1="0" x2="50" y2="1" width="0" layer="20" curve="90"/>
 <wire x1="1" y1="0" x2="0" y2="1" width="0" layer="20" curve="-90"/>
-<text x="17" y="46" size="2.54" layer="21" font="vector">probatio</text>
 <text x="27.09" y="19.42" size="1.27" layer="21" font="vector">SCL</text>
 <text x="27.01" y="16.33" size="1.27" layer="21" font="vector">SDA</text>
@@
 <text x="40.31" y="46.06" size="1.016" layer="22" font="vector" rot="MR270">SDA</text>
 <text x="37.67" y="46.04" size="1.016" layer="22" font="vector" rot="MR270">SCL</text>
-<text x="16.5" y="43.5" size="1.27" layer="21" font="vector">base-pcb v0_3_2</text>
+<text x="22.1" y="42.5" size="1.27" layer="21" font="vector">base-pcb v0_3_2</text>
 </plain>
 <attributes>
@@
 <element name="U$6" library="Batebit" package="1X04_SMD" value="M04WIRE_PAD" x="41" y="48.09" smashed="yes" rot="MR270"/>
 <element name="U$7" library="Batebit" package="1X04_SMD" value="M04WIRE_PAD" x="48.09" y="41" smashed="yes" rot="MR180"/>
-<element name="U$8" library="Batebit" package="1X04_SMD" value="M04WIRE_PAD" x="1.91" y="41" smashed="yes" rot="MR180"/>
+<element name="U$8" library="Batebit" package="1X04_SMD" value="M04WIRE_PAD" x="1.91" y="40.99" smashed="yes" rot="MR180"/>
 <element name="U$9" library="Batebit" package="1X04_SMD" value="M04WIRE_PAD" x="1.91" y="9" smashed="yes" rot="MR0"/>
-<element name="U$13" library="Batebit" package="BATEBIT_PEQ" value="BATEBIT_PEQ" x="24.88" y="24.25" smashed="yes" rot="MR0"/>
+<element name="U$13" library="Batebit" package="BATEBIT_PEQ" value="BATEBIT_PEQ" x="24.98" y="26.65" smashed="yes" rot="MR0"/>
+<element name="U$14" library="Batebit" package="PROBATIO" value="" x="25" y="44.7" smashed="yes"/>
 </elements>
 <signals>
@@
 <wire x1="3.2" y1="37.05" x2="3.2" y2="37.1" width="0.6096" layer="16"/>
 <wire x1="3.2" y1="37.1" x2="3.12" y2="37.18" width="0.6096" layer="16"/>
-<wire x1="3.12" y1="37.18" x2="1.91" y2="37.19" width="0.6096" layer="16"/>
+<wire x1="3.12" y1="37.18" x2="1.91" y2="37.18" width="0.6096" layer="16"/>
 <wire x1="30.36" y1="39.66" x2="37.4" y2="46.7" width="0.6096" layer="16"/>
 <wire x1="37.4" y1="46.7" x2="37.4" y2="47.88" width="0.6096" layer="16"/>
@@
 <wire x1="10.2" y1="48.02" x2="10.27" y2="48.09" width="0.6096" layer="16"/>
 <wire x1="16.61" y1="33.72" x2="16.61" y2="39.69" width="0.6096" layer="16"/>
-<wire x1="4.38" y1="39.72" x2="1.91" y2="39.73" width="0.6096" layer="16"/>
+<wire x1="4.38" y1="39.72" x2="1.91" y2="39.72" width="0.6096" layer="16"/>
 <wire x1="16.61" y1="33.72" x2="10.38" y2="33.72" width="0.6096" layer="16"/>
 <wire x1="10.38" y1="33.72" x2="4.38" y2="39.72" width="0.6096" layer="16"/>
@@
 <wire x1="4.7" y1="42.29" x2="4.7" y2="42.3" width="0.6096" layer="16"/>
 <wire x1="4.7" y1="42.3" x2="1.95" y2="42.3" width="0.6096" layer="16"/>
-<wire x1="1.95" y1="42.3" x2="1.91" y2="42.27" width="0.6096" layer="16"/>
+<wire x1="1.95" y1="42.3" x2="1.91" y2="42.26" width="0.6096" layer="16"/>
 <wire x1="36.63" y1="36.59" x2="36.63" y2="39.5" width="0.6096" layer="16"/>
 <wire x1="36.63" y1="39.5" x2="42.23" y2="45.1" width="0.6096" layer="16"/>
@@
 <wire x1="10.8" y1="39.2" x2="5.2" y2="44.8" width="0.6096" layer="16"/>
 <wire x1="5.2" y1="44.8" x2="5.19" y2="44.81" width="0.6096" layer="16"/>
-<wire x1="5.2" y1="44.8" x2="1.91" y2="44.81" width="0.6096" layer="16"/>
+<wire x1="5.2" y1="44.8" x2="1.91" y2="44.8" width="0.6096" layer="16"/>
 <wire x1="48.09" y1="44.81" x2="45.01" y2="44.81" width="0.6096" layer="16"/>
 <wire x1="39.4" y1="39.2" x2="45.01" y2="44.81" width="0.6096" layer="16"/>
